Commit message: need to test control

File: alphabot_simulator/alphabot_description/urdf/alphabot.xacro (robot description, xacro)
@@ -627,5 +627,5 @@
   <child link="camera_1"/>
 </joint>
-<joint name="Revolute 33" type="continuous">
+<joint name="Revolute 19" type="continuous">
   <origin xyz="0.0 -0.017 0.014953" rpy="0 0 0"/>
   <parent link="motor_1"/>

Commit message: need to tune pid controller, friction...

File: alphabot_simulator/alphabot_description/urdf/alphabot.xacro (robot description, xacro)
@@ -8,5 +8,5 @@
   <inertial>
     <origin xyz="-0.02 -1.94978353285355e-05 -0.00745233167839299" rpy="0 0 0"/>
-    <mass value="0.28642351470332406"/>
+    <mass value="0.2"/>
     <inertia ixx="0.000125" iyy="0.000266" izz="0.000389" ixy="-0.0" iyz="0.0" ixz="0.0"/>
   </inertial>
@@ -28,5 +28,5 @@
   <inertial>
     <origin xyz="-8.5543543531727e-08 -2.7755575615628914e-15 0.02005616243908092" rpy="0 0 0"/>
-    <mass value="0.005257224692902246"/>
+    <mass value="0.05"/>
     <inertia ixx="1e-06" iyy="1e-06" izz="0.0" ixy="-0.0" iyz="0.0" ixz="-0.0"/>
   </inertial>
@@ -48,5 +48,5 @@
   <inertial>
     <origin xyz="-8.554354357336036e-08 -2.7755575615628914e-15 0.02005616243908092" rpy="0 0 0"/>
-    <mass value="0.005257224692902246"/>
+    <mass value="0.05"/>
     <inertia ixx="1e-06" iyy="1e-06" izz="0.0" ixy="-0.0" iyz="0.0" ixz="-0.0"/>
   </inertial>
@@ -68,5 +68,5 @@
   <inertial>
     <origin xyz="8.554362089518985e-08 -2.7824964554667986e-15 0.020056162439080885" rpy="0 0 0"/>
-    <mass value="0.005257224692902246"/>
+    <mass value="0.05"/>
     <inertia ixx="1e-06" iyy="1e-06" izz="0.0" ixy="-0.0" iyz="0.0" ixz="-0.0"/>
   </inertial>
@@ -88,5 +88,5 @@
   <inertial>
     <origin xyz="8.554362092988432e-08 -2.7408630920433552e-15 0.020056162439080885" rpy="0 0 0"/>
-    <mass value="0.005257224692902246"/>
+    <mass value="0.05"/>
     <inertia ixx="1e-06" iyy="1e-06" izz="0.0" ixy="-0.0" iyz="0.0" ixz="-0.0"/>
   </inertial>
@@ -128,5 +128,5 @@
   <inertial>
     <origin xyz="1.5959455978986625e-16 -0.024725409875466932 -3.316783929825304e-07" rpy="0 0 0"/>
-    <mass value="0.06207035736097537"/>
+    <mass value="0.2"/>
     <inertia ixx="1.3e-05" iyy="2e-06" izz="1.3e-05" ixy="0.0" iyz="-0.0" ixz="0.0"/>
   </inertial>
@@ -148,5 +148,5 @@
   <inertial>
     <origin xyz="1.6653345369377348e-16 0.024725409875466935 -3.3167839298513246e-07" rpy="0 0 0"/>
-    <mass value="0.06207035736097537"/>
+    <mass value="0.2"/>
     <inertia ixx="1.3e-05" iyy="2e-06" izz="1.3e-05" ixy="-0.0" iyz="-0.0" ixz="-0.0"/>
   </inertial>
@@ -188,5 +188,5 @@
   <inertial>
     <origin xyz="-5.612034448265746e-11 -0.004604091884807676 0.014952668255257739" rpy="0 0 0"/>
-    <mass value="0.006835989534703237"/>
+    <mass value="0.05"/>
     <inertia ixx="0.0" iyy="0.0" izz="0.0" ixy="-0.0" iyz="0.0" ixz="0.0"/>
   </inertial>
@@ -208,5 +208,5 @@
   <inertial>
     <origin xyz="5.6120341013210506e-11 0.04460409188480768 0.014952668255257739" rpy="0 0 0"/>
-    <mass value="0.006835989534703237"/>
+    <mass value="0.05"/>
     <inertia ixx="0.0" iyy="0.0" izz="0.0" ixy="-0.0" iyz="-0.0" ixz="-0.0"/>
   </inertial>
@@ -580,4 +580,5 @@
   <child link="left_wheel_1"/>
   <axis xyz="0.0 1.0 0.0"/>
+  <dynamics damping="2.0" friction="2.0"/>
 </joint>
 <joint name="Rigid 20" type="fixed">
@@ -616,4 +617,6 @@
   <child link="servo_2_1"/>
   <axis xyz="0.0 1.0 0.0"/>
+  <dynamics damping="0.1" friction="100"/>
+  <limit effort="130" lower="-1.57" upper="1.57" velocity="6.98"/>
 </joint>
 <joint name="Revolute 31" type="continuous">
@@ -622,4 +625,6 @@
   <child link="servo_1_1"/>
   <axis xyz="-0.0 -0.0 1.0"/>
+  <dynamics damping="0.01" friction="1"/>
+  <limit effort="130" lower="-1.57" upper="1.57" velocity="6.98"/>
 </joint>
 <joint name="Rigid 32" type="fixed">
@@ -633,4 +638,5 @@
   <child link="right_wheel_1"/>
   <axis xyz="0.0 1.0 -0.0"/>
+  <dynamics damping="2.0" friction="2.0"/>
 </joint>
 <joint name="Rigid 43" type="fixed">

Commit message: update, robot still drifts

File: alphabot_simulator/alphabot_description/urdf/alphabot.xacro (robot description, xacro)
@@ -5,9 +5,8 @@
 <xacro:include filename="$(find alphabot_description)/urdf/alphabot.gazebo" />
 <link name="base_link">
-  <pose> 0 0 0 0 0 0 </pose>
-  <inertial>
-    <origin xyz="-0.02 -1.94978353285355e-05 -0.00745233167839299" rpy="0 0 0"/>
+  <inertial>
+    <origin xyz="3.9964129120210354e-17 -1.949783532853795e-05 0.014547668321607015" rpy="0 0 0"/>
     <mass value="0.2"/>
-    <inertia ixx="0.000125" iyy="0.000266" izz="0.000389" ixy="-0.0" iyz="0.0" ixz="0.0"/>
+    <inertia ixx="0.000125" iyy="0.000266" izz="0.000389" ixy="-0.0" iyz="-0.0" ixz="0.0"/>
   </inertial>
   <visual>
@@ -27,10 +26,10 @@
 <link name="spacer_1_1">
   <inertial>
-    <origin xyz="-8.5543543531727e-08 -2.7755575615628914e-15 0.02005616243908092" rpy="0 0 0"/>
+    <origin xyz="-8.554354349876725e-08 -2.7824964554667986e-15 0.020056162439080906" rpy="0 0 0"/>
     <mass value="0.05"/>
     <inertia ixx="1e-06" iyy="1e-06" izz="0.0" ixy="-0.0" iyz="0.0" ixz="-0.0"/>
   </inertial>
   <visual>
-    <origin xyz="-0.008948 -0.04191 0.004952" rpy="0 0 0"/>
+    <origin xyz="-0.028948 -0.04191 -0.017048" rpy="0 0 0"/>
     <geometry>
       <mesh filename="package://alphabot_description/meshes/spacer_1_1.stl" scale="0.001 0.001 0.001"/>
@@ -39,5 +38,5 @@
   </visual>
   <collision>
-    <origin xyz="-0.008948 -0.04191 0.004952" rpy="0 0 0"/>
+    <origin xyz="-0.028948 -0.04191 -0.017048" rpy="0 0 0"/>
     <geometry>
       <mesh filename="package://alphabot_description/meshes/spacer_1_1.stl" scale="0.001 0.001 0.001"/>
@@ -47,10 +46,10 @@
 <link name="spacer_1_2">
   <inertial>
-    <origin xyz="-8.554354357336036e-08 -2.7755575615628914e-15 0.02005616243908092" rpy="0 0 0"/>
+    <origin xyz="-8.554354354040061e-08 -2.7755575615628914e-15 0.020056162439080906" rpy="0 0 0"/>
     <mass value="0.05"/>
     <inertia ixx="1e-06" iyy="1e-06" izz="0.0" ixy="-0.0" iyz="0.0" ixz="-0.0"/>
   </inertial>
   <visual>
-    <origin xyz="-0.008948 0.04191 0.004952" rpy="0 0 0"/>
+    <origin xyz="-0.028948 0.04191 -0.017048" rpy="0 0 0"/>
     <geometry>
       <mesh filename="package://alphabot_description/meshes/spacer_1_2.stl" scale="0.001 0.001 0.001"/>
@@ -59,5 +58,5 @@
   </visual>
   <collision>
-    <origin xyz="-0.008948 0.04191 0.004952" rpy="0 0 0"/>
+    <origin xyz="-0.028948 0.04191 -0.017048" rpy="0 0 0"/>
     <geometry>
       <mesh filename="package://alphabot_description/meshes/spacer_1_2.stl" scale="0.001 0.001 0.001"/>
@@ -67,10 +66,10 @@
 <link name="spacer_1_3">
   <inertial>
-    <origin xyz="8.554362089518985e-08 -2.7824964554667986e-15 0.020056162439080885" rpy="0 0 0"/>
+    <origin xyz="8.554362094723156e-08 -2.7824964554667986e-15 0.02005616243908087" rpy="0 0 0"/>
     <mass value="0.05"/>
     <inertia ixx="1e-06" iyy="1e-06" izz="0.0" ixy="-0.0" iyz="0.0" ixz="-0.0"/>
   </inertial>
   <visual>
-    <origin xyz="0.048948 0.04191 0.004952" rpy="0 0 0"/>
+    <origin xyz="0.028948 0.04191 -0.017048" rpy="0 0 0"/>
     <geometry>
       <mesh filename="package://alphabot_description/meshes/spacer_1_3.stl" scale="0.001 0.001 0.001"/>
@@ -79,5 +78,5 @@
   </visual>
   <collision>
-    <origin xyz="0.048948 0.04191 0.004952" rpy="0 0 0"/>
+    <origin xyz="0.028948 0.04191 -0.017048" rpy="0 0 0"/>
     <geometry>
       <mesh filename="package://alphabot_description/meshes/spacer_1_3.stl" scale="0.001 0.001 0.001"/>
@@ -87,10 +86,10 @@
 <link name="spacer_1_4">
   <inertial>
-    <origin xyz="8.554362092988432e-08 -2.7408630920433552e-15 0.020056162439080885" rpy="0 0 0"/>
+    <origin xyz="8.554362097498713e-08 -2.7478019859472624e-15 0.02005616243908087" rpy="0 0 0"/>
     <mass value="0.05"/>
     <inertia ixx="1e-06" iyy="1e-06" izz="0.0" ixy="-0.0" iyz="0.0" ixz="-0.0"/>
   </inertial>
   <visual>
-    <origin xyz="0.048948 -0.04191 0.004952" rpy="0 0 0"/>
+    <origin xyz="0.028948 -0.04191 -0.017048" rpy="0 0 0"/>
     <geometry>
       <mesh filename="package://alphabot_description/meshes/spacer_1_4.stl" scale="0.001 0.001 0.001"/>
@@ -99,5 +98,5 @@
   </visual>
   <collision>
-    <origin xyz="0.048948 -0.04191 0.004952" rpy="0 0 0"/>
+    <origin xyz="0.028948 -0.04191 -0.017048" rpy="0 0 0"/>
     <geometry>
       <mesh filename="package://alphabot_description/meshes/spacer_1_4.stl" scale="0.001 0.001 0.001"/>
@@ -107,10 +106,10 @@
 <link name="ultasonic_1">
   <inertial>
-    <origin xyz="0.033193707682986025 0.019999904709901414 0.01996218206000405" rpy="0 0 0"/>
+    <origin xyz="0.033193707682986046 -9.529009860237083e-08 -0.0020378179399959465" rpy="0 0 0"/>
     <mass value="0.02930398813229992"/>
     <inertia ixx="6e-06" iyy="1e-06" izz="5e-06" ixy="-0.0" iyz="0.0" ixz="-0.0"/>
   </inertial>
   <visual>
-    <origin xyz="0.02 0.02 0.014905" rpy="0 0 0"/>
+    <origin xyz="-0.0 -0.0 -0.029095" rpy="0 0 0"/>
     <geometry>
       <mesh filename="package://alphabot_description/meshes/ultasonic_1.stl" scale="0.001 0.001 0.001"/>
@@ -119,5 +118,5 @@
   </visual>
   <collision>
-    <origin xyz="0.02 0.02 0.014905" rpy="0 0 0"/>
+    <origin xyz="-0.0 -0.0 -0.029095" rpy="0 0 0"/>
     <geometry>
       <mesh filename="package://alphabot_description/meshes/ultasonic_1.stl" scale="0.001 0.001 0.001"/>
@@ -127,10 +126,10 @@
 <link name="AA_1">
   <inertial>
-    <origin xyz="1.5959455978986625e-16 -0.024725409875466932 -3.316783929825304e-07" rpy="0 0 0"/>
+    <origin xyz="1.7694179454963432e-16 -0.024725409875466925 -3.3167839298339774e-07" rpy="0 0 0"/>
     <mass value="0.2"/>
     <inertia ixx="1.3e-05" iyy="2e-06" izz="1.3e-05" ixy="0.0" iyz="-0.0" ixz="0.0"/>
   </inertial>
   <visual>
-    <origin xyz="0.04225 -0.026 -0.004048" rpy="0 0 0"/>
+    <origin xyz="0.02225 -0.026 -0.026048" rpy="0 0 0"/>
     <geometry>
       <mesh filename="package://alphabot_description/meshes/AA_1.stl" scale="0.001 0.001 0.001"/>
@@ -139,5 +138,5 @@
   </visual>
   <collision>
-    <origin xyz="0.04225 -0.026 -0.004048" rpy="0 0 0"/>
+    <origin xyz="0.02225 -0.026 -0.026048" rpy="0 0 0"/>
     <geometry>
       <mesh filename="package://alphabot_description/meshes/AA_1.stl" scale="0.001 0.001 0.001"/>
@@ -147,10 +146,10 @@
 <link name="AA_2">
   <inertial>
-    <origin xyz="1.6653345369377348e-16 0.024725409875466935 -3.3167839298513246e-07" rpy="0 0 0"/>
+    <origin xyz="2.0816681711721685e-16 0.024725409875466935 -3.3167839298339774e-07" rpy="0 0 0"/>
     <mass value="0.2"/>
     <inertia ixx="1.3e-05" iyy="2e-06" izz="1.3e-05" ixy="-0.0" iyz="-0.0" ixz="-0.0"/>
   </inertial>
   <visual>
-    <origin xyz="0.05775 0.026 -0.004048" rpy="0 0 0"/>
+    <origin xyz="0.03775 0.026 -0.026048" rpy="0 0 0"/>
     <geometry>
       <mesh filename="package://alphabot_description/meshes/AA_2.stl" scale="0.001 0.001 0.001"/>
@@ -159,5 +158,5 @@
   </visual>
   <collision>
-    <origin xyz="0.05775 0.026 -0.004048" rpy="0 0 0"/>
+    <origin xyz="0.03775 0.026 -0.026048" rpy="0 0 0"/>
     <geometry>
       <mesh filename="package://alphabot_description/meshes/AA_2.stl" scale="0.001 0.001 0.001"/>
@@ -167,10 +166,10 @@
 <link name="battery_case_1">
   <inertial>
-    <origin xyz="-0.030001214328793952 0.019965972372322435 0.013658871061547454" rpy="0 0 0"/>
+    <origin xyz="-0.030001214328793938 -3.4027627677573753e-05 -0.008341128938452552" rpy="0 0 0"/>
     <mass value="0.06781923232527433"/>
     <inertia ixx="2.2e-05" iyy="8e-06" izz="2.8e-05" ixy="-0.0" iyz="0.0" ixz="0.0"/>
   </inertial>
   <visual>
-    <origin xyz="0.02 0.02 0.014905" rpy="0 0 0"/>
+    <origin xyz="-0.0 -0.0 -0.029095" rpy="0 0 0"/>
     <geometry>
       <mesh filename="package://alphabot_description/meshes/battery_case_1.stl" scale="0.001 0.001 0.001"/>
@@ -179,5 +178,5 @@
   </visual>
   <collision>
-    <origin xyz="0.02 0.02 0.014905" rpy="0 0 0"/>
+    <origin xyz="-0.0 -0.0 -0.029095" rpy="0 0 0"/>
     <geometry>
       <mesh filename="package://alphabot_description/meshes/battery_case_1.stl" scale="0.001 0.001 0.001"/>
@@ -187,10 +186,10 @@
 <link name="motor_1">
   <inertial>
-    <origin xyz="-5.612034448265746e-11 -0.004604091884807676 0.014952668255257739" rpy="0 0 0"/>
+    <origin xyz="-5.612031395152428e-11 -0.024604091884807677 -0.007047331744742258" rpy="0 0 0"/>
     <mass value="0.05"/>
     <inertia ixx="0.0" iyy="0.0" izz="0.0" ixy="-0.0" iyz="0.0" ixz="0.0"/>
   </inertial>
   <visual>
-    <origin xyz="0.02 0.02 0.014905" rpy="0 0 0"/>
+    <origin xyz="-0.0 -0.0 -0.029095" rpy="0 0 0"/>
     <geometry>
       <mesh filename="package://alphabot_description/meshes/motor_1.stl" scale="0.001 0.001 0.001"/>
@@ -199,5 +198,5 @@
   </visual>
   <collision>
-    <origin xyz="0.02 0.02 0.014905" rpy="0 0 0"/>
+    <origin xyz="-0.0 -0.0 -0.029095" rpy="0 0 0"/>
     <geometry>
       <mesh filename="package://alphabot_description/meshes/motor_1.stl" scale="0.001 0.001 0.001"/>
@@ -207,10 +206,10 @@
 <link name="motor_2">
   <inertial>
-    <origin xyz="5.6120341013210506e-11 0.04460409188480768 0.014952668255257739" rpy="0 0 0"/>
+    <origin xyz="5.6120382785351805e-11 0.024604091884807677 -0.007047331744742258" rpy="0 0 0"/>
     <mass value="0.05"/>
     <inertia ixx="0.0" iyy="0.0" izz="0.0" ixy="-0.0" iyz="-0.0" ixz="-0.0"/>
   </inertial>
   <visual>
-    <origin xyz="0.02 0.02 0.014905" rpy="0 0 0"/>
+    <origin xyz="-0.0 -0.0 -0.029095" rpy="0 0 0"/>
     <geometry>
       <mesh filename="package://alphabot_description/meshes/motor_2.stl" scale="0.001 0.001 0.001"/>
@@ -219,5 +218,5 @@
   </visual>
   <collision>
-    <origin xyz="0.02 0.02 0.014905" rpy="0 0 0"/>
+    <origin xyz="-0.0 -0.0 -0.029095" rpy="0 0 0"/>
     <geometry>
       <mesh filename="package://alphabot_description/meshes/motor_2.stl" scale="0.001 0.001 0.001"/>
@@ -225,32 +224,12 @@
   </collision>
 </link>
-<link name="left_wheel_1">
-  <inertial>
-    <origin xyz="-3.6085538349002466e-06 0.006410625405004984 -2.519122826068395e-06" rpy="0 0 0"/>
-    <mass value="0.10619619440264885"/>
-    <inertia ixx="1.8e-05" iyy="3.1e-05" izz="1.8e-05" ixy="-0.0" iyz="-0.0" ixz="0.0"/>
-  </inertial>
-  <visual>
-    <origin xyz="0.02 -0.037 -4.8e-05" rpy="0 0 0"/>
-    <geometry>
-      <mesh filename="package://alphabot_description/meshes/left_wheel_1.stl" scale="0.001 0.001 0.001"/>
-    </geometry>
-    <material name="black"/>
-  </visual>
-  <collision>
-    <origin xyz="0.02 -0.037 -4.8e-05" rpy="0 0 0"/>
-    <geometry>
-      <mesh filename="package://alphabot_description/meshes/left_wheel_1.stl" scale="0.001 0.001 0.001"/>
-    </geometry>
-  </collision>
-</link>
 <link name="top_link_1">
   <inertial>
-    <origin xyz="0.02896008554358224 0.04191000000000044 0.0024996683216068558" rpy="0 0 0"/>
+    <origin xyz="0.028960085543582276 0.04191000000000044 0.0024996683216068558" rpy="0 0 0"/>
     <mass value="0.37189545514665234"/>
     <inertia ixx="0.000281" iyy="0.000282" izz="0.000561" ixy="0.0" iyz="-0.0" ixz="0.0"/>
   </inertial>
   <visual>
-    <origin xyz="0.048948 0.04191 -0.035423" rpy="0 0 0"/>
+    <origin xyz="0.028948 0.04191 -0.057423" rpy="0 0 0"/>
     <geometry>
       <mesh filename="package://alphabot_description/meshes/top_link_1.stl" scale="0.001 0.001 0.001"/>
@@ -259,5 +238,5 @@
   </visual>
   <collision>
-    <origin xyz="0.048948 0.04191 -0.035423" rpy="0 0 0"/>
+    <origin xyz="0.028948 0.04191 -0.057423" rpy="0 0 0"/>
     <geometry>
       <mesh filename="package://alphabot_description/meshes/top_link_1.stl" scale="0.001 0.001 0.001"/>
@@ -267,17 +246,17 @@
 <link name="pantilt_1_1">
   <inertial>
-    <origin xyz="-0.003632741722051625 -2.87666307189565e-15 0.0018087943330409445" rpy="0 0 0"/>
+    <origin xyz="-0.0036327417220515914 -2.873247422695575e-15 0.0018087943330409653" rpy="0 0 0"/>
     <mass value="0.02484644401179895"/>
     <inertia ixx="2e-06" iyy="3e-06" izz="5e-06" ixy="0.0" iyz="-0.0" ixz="-0.0"/>
   </inertial>
   <visual>
-    <origin xyz="0.019988 0.0 -0.040423" rpy="0 0 0"/>
+    <origin xyz="-1.2e-05 0.0 -0.062423" rpy="0 0 0"/>
     <geometry>
       <mesh filename="package://alphabot_description/meshes/pantilt_1_1.stl" scale="0.001 0.001 0.001"/>
     </geometry>
-    <material name="black"/>
-  </visual>
-  <collision>
-    <origin xyz="0.019988 0.0 -0.040423" rpy="0 0 0"/>
+    <material name="blue"/>
+  </visual>
+  <collision>
+    <origin xyz="-1.2e-05 0.0 -0.062423" rpy="0 0 0"/>
     <geometry>
       <mesh filename="package://alphabot_description/meshes/pantilt_1_1.stl" scale="0.001 0.001 0.001"/>
@@ -287,10 +266,10 @@
 <link name="servo_emax_1_1">
   <inertial>
-    <origin xyz="8.554358225595915e-08 1.2546002784527504e-13 0.0035263014079521676" rpy="0 0 0"/>
+    <origin xyz="8.554358228704865e-08 1.254629415068201e-13 0.0035263014079521815" rpy="0 0 0"/>
     <mass value="0.0035428307305659244"/>
     <inertia ixx="0.0" iyy="0.0" izz="0.0" ixy="-0.0" iyz="-0.0" ixz="0.0"/>
   </inertial>
   <visual>
-    <origin xyz="0.019988 0.0 -0.042423" rpy="0 0 0"/>
+    <origin xyz="-1.2e-05 0.0 -0.064423" rpy="0 0 0"/>
     <geometry>
       <mesh filename="package://alphabot_description/meshes/servo_emax_1_1.stl" scale="0.001 0.001 0.001"/>
@@ -299,5 +278,5 @@
   </visual>
   <collision>
-    <origin xyz="0.019988 0.0 -0.042423" rpy="0 0 0"/>
+    <origin xyz="-1.2e-05 0.0 -0.064423" rpy="0 0 0"/>
     <geometry>
       <mesh filename="package://alphabot_description/meshes/servo_emax_1_1.stl" scale="0.001 0.001 0.001"/>
@@ -307,10 +286,10 @@
 <link name="pantilt_2_1">
   <inertial>
-    <origin xyz="-0.024434540776768092 0.058954045810892274 0.003603404587610895" rpy="0 0 0"/>
+    <origin xyz="-0.0044345407767680915 0.08095404581089227 0.003603404587610881" rpy="0 0 0"/>
     <mass value="0.05139456940551715"/>
     <inertia ixx="1e-05" iyy="1.1e-05" izz="1.4e-05" ixy="-0.0" iyz="-0.0" ixz="-2e-06"/>
   </inertial>
   <visual>
-    <origin xyz="-0.01175 0.059723 -0.069723" rpy="0 0 0"/>
+    <origin xyz="-0.01175 0.081723 -0.091723" rpy="0 0 0"/>
     <geometry>
       <mesh filename="package://alphabot_description/meshes/pantilt_2_1.stl" scale="0.001 0.001 0.001"/>
@@ -319,5 +298,5 @@
   </visual>
   <collision>
-    <origin xyz="-0.01175 0.059723 -0.069723" rpy="0 0 0"/>
+    <origin xyz="-0.01175 0.081723 -0.091723" rpy="0 0 0"/>
     <geometry>
       <mesh filename="package://alphabot_description/meshes/pantilt_2_1.stl" scale="0.001 0.001 0.001"/>
@@ -327,10 +306,10 @@
 <link name="servo_emax_2_1">
   <inertial>
-    <origin xyz="-0.0919834516518788 -0.021846169429072 -0.04697233167823213" rpy="0 0 0"/>
+    <origin xyz="-0.09208845165187876 -0.04184616942907199 -0.06897233167823215" rpy="0 0 0"/>
     <mass value="0.0026502814230264554"/>
     <inertia ixx="0.0" iyy="0.0" izz="0.0" ixy="-0.0" iyz="-0.0" ixz="-0.0"/>
   </inertial>
   <visual>
-    <origin xyz="-0.098148 -0.005389 -0.136545" rpy="0 0 0"/>
+    <origin xyz="-0.118253 -0.025389 -0.180545" rpy="0 0 0"/>
     <geometry>
       <mesh filename="package://alphabot_description/meshes/servo_emax_2_1.stl" scale="0.001 0.001 0.001"/>
@@ -339,5 +318,5 @@
   </visual>
   <collision>
-    <origin xyz="-0.098148 -0.005389 -0.136545" rpy="0 0 0"/>
+    <origin xyz="-0.118253 -0.025389 -0.180545" rpy="0 0 0"/>
     <geometry>
       <mesh filename="package://alphabot_description/meshes/servo_emax_2_1.stl" scale="0.001 0.001 0.001"/>
@@ -347,10 +326,10 @@
 <link name="pantilt_3_1">
   <inertial>
-    <origin xyz="0.11125626443826739 -0.013095879873687063 0.0004311932686931613" rpy="0 0 0"/>
+    <origin xyz="0.13325626443826744 -0.013095879873687058 0.02043119326869315" rpy="0 0 0"/>
     <mass value="0.025707768034284914"/>
     <inertia ixx="6e-06" iyy="3e-06" izz="4e-06" ixy="0.0" iyz="0.0" ixz="-0.0"/>
   </inertial>
   <visual>
-    <origin xyz="0.096261 -0.0148 -0.100061" rpy="0 0 0"/>
+    <origin xyz="0.098261 -0.0148 -0.102061" rpy="0 0 0"/>
     <geometry>
       <mesh filename="package://alphabot_description/meshes/pantilt_3_1.stl" scale="0.001 0.001 0.001"/>
@@ -359,5 +338,5 @@
   </visual>
   <collision>
-    <origin xyz="0.096261 -0.0148 -0.100061" rpy="0 0 0"/>
+    <origin xyz="0.098261 -0.0148 -0.102061" rpy="0 0 0"/>
     <geometry>
       <mesh filename="package://alphabot_description/meshes/pantilt_3_1.stl" scale="0.001 0.001 0.001"/>
@@ -367,17 +346,17 @@
 <link name="servo_2_1">
   <inertial>
-    <origin xyz="8.554358096879433e-08 0.012439350245232206 0.005558642662359295" rpy="0 0 0"/>
+    <origin xyz="8.55435810034888e-08 0.012439350245232213 0.005558642662359281" rpy="0 0 0"/>
     <mass value="0.048166128445804444"/>
     <inertia ixx="4e-06" iyy="3e-06" izz="3e-06" ixy="-0.0" iyz="-0.0" ixz="-0.0"/>
   </inertial>
   <visual>
-    <origin xyz="-0.007112 0.0112 -0.089573" rpy="0 0 0"/>
+    <origin xyz="-0.027112 0.0112 -0.111573" rpy="0 0 0"/>
     <geometry>
       <mesh filename="package://alphabot_description/meshes/servo_2_1.stl" scale="0.001 0.001 0.001"/>
     </geometry>
-    <material name="light_blue"/>
-  </visual>
-  <collision>
-    <origin xyz="-0.007112 0.0112 -0.089573" rpy="0 0 0"/>
+    <material name="silver"/>
+  </visual>
+  <collision>
+    <origin xyz="-0.027112 0.0112 -0.111573" rpy="0 0 0"/>
     <geometry>
       <mesh filename="package://alphabot_description/meshes/servo_2_1.stl" scale="0.001 0.001 0.001"/>
@@ -387,10 +366,10 @@
 <link name="servo_1_1">
   <inertial>
-    <origin xyz="0.005559059884334831 -1.4899192990469603e-15 0.012439018566839377" rpy="0 0 0"/>
+    <origin xyz="0.005559059884334861 -1.4876988529977098e-15 0.012439018566839363" rpy="0 0 0"/>
     <mass value="0.048166128445804444"/>
     <inertia ixx="3e-06" iyy="4e-06" izz="3e-06" ixy="-0.0" iyz="-0.0" ixz="-0.0"/>
   </inertial>
   <visual>
-    <origin xyz="0.019988 0.0 -0.051923" rpy="0 0 0"/>
+    <origin xyz="-1.2e-05 0.0 -0.073923" rpy="0 0 0"/>
     <geometry>
       <mesh filename="package://alphabot_description/meshes/servo_1_1.stl" scale="0.001 0.001 0.001"/>
@@ -399,5 +378,5 @@
   </visual>
   <collision>
-    <origin xyz="0.019988 0.0 -0.051923" rpy="0 0 0"/>
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