Commit message: fix base link

File: alphabot_simulator/alphabot_description/urdf/alphabot.xacro (robot description, xacro)
@@ -2,6 +2,5 @@
 <robot name="alphabot" xmlns:xacro="http://www.ros.org/wiki/xacro">
 <xacro:include filename="$(find alphabot_description)/urdf/materials.xacro" />
-<xacro:include filename="$(find alphabot_description)/urdf/alphabot.trans" />
-<xacro:include filename="$(find alphabot_description)/urdf/alphabot.gazebo" />
+<link name="base_footprint" />
 <link name="base_link">
   <inertial>
@@ -355,5 +354,5 @@
       <mesh filename="package://alphabot_description/meshes/servo_2_1.stl" scale="0.001 0.001 0.001"/>
     </geometry>
-    <material name="silver"/>
+    <material name="light_blue"/>
   </visual>
   <collision>
@@ -524,4 +523,8 @@
   </collision>
 </link>
+<joint name="base_footprint_joint" type="fixed">
+  <parent link="base_footprint" />
+  <child link="base_link" />
+</joint>
 <joint name="Rigid 6" type="fixed">
   <origin xyz="0.028948 0.04191 0.017048" rpy="0 0 0"/>
@@ -609,6 +612,4 @@
   <child link="servo_2_1"/>
   <axis xyz="0.0 1.0 0.0"/>
-  <dynamics damping="0.1" friction="100"/>
-  <limit effort="130" lower="-1.57" upper="1.57" velocity="6.98"/>
 </joint>
 <joint name="Revolute 31" type="continuous">
@@ -617,6 +618,4 @@
   <child link="servo_1_1"/>
   <axis xyz="-0.0 -0.0 1.0"/>
-  <dynamics damping="0.01" friction="1"/>
-  <limit effort="130" lower="-1.57" upper="1.57" velocity="6.98"/>
 </joint>
 <joint name="Rigid 32" type="fixed">
@@ -650,5 +649,4 @@
   <child link="left_wheel_1"/>
   <axis xyz="0.0 1.0 -0.0"/>
-  <dynamics damping="2" friction="2"/>
 </joint>
 <joint name="Revolute 19" type="continuous">
@@ -657,5 +655,4 @@
   <child link="right_wheel_1"/>
   <axis xyz="0.0 1.0 -0.0"/>
-  <dynamics damping="2" friction="2"/>
 </joint>
 </robot>
